File: kitcat/Projeto2025.2/Projeto2025.2.kicad_pcb (KiCad board)
At the start: 2 copper layers, 23 parts, among them IC1 LA4182, J1 Conn_01x02, J2 Conn_01x02, J3 Conn_01x02, J4 Conn_01x02, J5 Conn_01x02

Commit message: aaaaa
Parts:
- moved J4 75.4 mm to (193.3, 67.5), turned to 90 degrees
- moved J2 69.5 mm to (186.7, 99.7), turned to 180 degrees
- moved D1 64.4 mm to (184.5, 63.5), turned to 90 degrees
- moved RV1 60.8 mm to (181.5, 112.5)
- moved C9 57.1 mm to (187.0, 91.0), turned to 90 degrees
- moved C12 53.7 mm to (187.5, 78.5), turned to 180 degrees
- moved J1 52.7 mm to (159.7, 101.8), turned to -90 degrees
- moved C11 52.5 mm to (186.5, 70.0), turned to 90 degrees
- moved J5 52.3 mm to (162.2, 67.7), turned to 180 degrees
- moved J3 52.0 mm to (165.0, 112.5), turned to -90 degrees
- moved C10 50.9 mm to (181.0, 78.5), turned to -90 degrees
- moved C6 47.5 mm to (172.5, 97.5), turned to 180 degrees
- moved R1 47.0 mm to (179.5, 65.5), turned to 90 degrees
- moved C2 38.1 mm to (163.0, 83.0)
- moved C7 36.2 mm to (173.0, 66.0)
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Connections:
- C1 pad 2: Net-(J1-Pin_2) -> Net-(J1-Pin_1)
- J1 pad 1: GNDREF -> Net-(J1-Pin_1)
- J1 pad 2: Net-(J1-Pin_2) -> GNDREF
- J3 pad 1: Net-(J3-Pin_1) -> GNDREF
- J3 pad 2: GNDREF -> Net-(J3-Pin_2)
- J5 pad 1: GNDREF -> Net-(IC1-12/VCC)
- J5 pad 2: Net-(IC1-12/VCC) -> GNDREF
- RV1 pad 1: Net-(J3-Pin_1) -> Net-(J3-Pin_2)
Routing:
- net GNDREF: track 0.00 -> 44.0 mm
- net Net-(C5-Pad1): track 0.00 -> 32.7 mm
- net Net-(IC1-12/VCC): track 0.00 -> 27.0 mm
- net Net-(J1-Pin_1): track 0.00 -> 26.3 mm
- net Net-(IC1-8/IN1): track 0.00 -> 18.2 mm
- net Net-(J2-Pin_2): track 0.00 -> 17.0 mm
- net Net-(IC1-2/OUT2): track 0.00 -> 16.6 mm
- net Net-(IC1-11/OUT1): track 0.00 -> 15.8 mm
- net Net-(C8-Pad1): track 0.00 -> 14.4 mm
- net Net-(J3-Pin_2): track 0.00 -> 11.8 mm
- net Net-(J4-Pin_1): track 0.00 -> 10.3 mm
- net Net-(IC1-6/DC): track 0.00 -> 6.51 mm
- net Net-(IC1-3/BS2): track 0.00 -> 6.38 mm
- net Net-(D1-Pad2): track 0.00 -> 5.75 mm
- net Net-(IC1-5/IN2): track 0.00 -> 5.51 mm
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- added copper zone on B.Cu, net GNDREF
Other:
- board outline added: 52 x 61.5 mm
