File: kitcat/Projeto2025.2/Projeto2025.2.kicad_sch (KiCad schematic)
At the start: 23 parts, among them IC1 LA4182, J1 Conn_01x02, J2 Conn_01x02, J3 Conn_01x02, J4 Conn_01x02, J5 Conn_01x02

Commit message: Update Projeto2025.2.kicad_sch
Parts:
- C11: value 100nF -> 150nF
Changed lines of the file:
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@@
 			)
 		)
-		(property "Value" "100nF"
+		(property "Value" "150nF"
 			(at 187.96 104.1399 0)
 			(effects

Commit message: s
Parts:
- C1, C12: footprint Capacitor_THT:CP_Radial_D10.0mm_P5.00mm -> aavirk:Capacitor_Eletrolítico_7.5mm
- C10, C4, C6, C9: footprint Capacitor_THT:CP_Radial_D10.0mm_P5.00mm -> aavirk:Capacitor_Eletrolítico_5mm
- C11, C3: footprint (none) -> aavirk:Capacitor_Poliesterp
- C2: footprint (none) -> aavirk:Capacitor_Eletrolítico_5mm
- C5, C8: footprint (none) -> aavirk:Capacitor_Poliesterg
- C7: footprint Capacitor_THT:CP_Radial_D10.0mm_P5.00mm -> aavirk:Capacitor_Eletrolítico_10mm
- D1: footprint LED_THT:LED_D5.0mm -> aavirk:Led_5mm
- IC1: footprint Virk:LA4182 -> aavirk:Circuito integrado
- J1, J2, J3, J4, J5: footprint (none) -> aavirk:Conector KRE
- R1: footprint (none) -> aavirk:Resistor_220_1_4W
- R2, R3: footprint (none) -> aavirk:Resistor_1_4W
- RV1: footprint (none) -> aavirk:Potenciometro_dual
Connections:
- net GNDREF: now also C7.2, D1.1, J5.1 (Pin_1)
Changed lines of the file:
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@@
+	)
+	(junction
+		(at 189.23 68.58)
+		(diameter 0)
+		(color 0 0 0 0)
 	)
 	(junction
@@
 	(wire
 		(pts
+			(xy 189.23 68.58) (xy 198.12 68.58)
+		)
+		(stroke
+			(width 0)
+			(type default)
+		)
+	)
+	(wire
+		(pts
 			(xy 184.15 77.47) (xy 184.15 83.82)
 		)
@@
 	(wire
 		(pts
-			(xy 185.42 68.58) (xy 198.12 68.58)
+			(xy 185.42 68.58) (xy 189.23 68.58)
 		)
 		(stroke
@@
 			)
 		)
-		(property "Footprint" "Capacitor_THT:CP_Radial_D10.0mm_P5.00mm"
+		(property "Footprint" "aavirk:Capacitor_Eletrolítico_5mm"
 			(at 106.3752 106.68 0)
 			(effects
@@
 			)
 		)
-		(property "Footprint" "Capacitor_THT:CP_Radial_D10.0mm_P5.00mm"
+		(property "Footprint" "aavirk:Capacitor_Eletrolítico_5mm"
 			(at 168.6052 106.68 0)
 			(effects
@@
 			)
 		)
-		(property "Footprint" ""
+		(property "Footprint" "aavirk:Conector KRE"
 			(at 220.98 60.96 0)
 			(effects
@@
 			)
 		)
-		(property "Footprint" ""
+		(property "Footprint" "aavirk:Conector KRE"
 			(at 53.34 96.52 0)
 			(effects
@@
 			)
 		)
-		(property "Footprint" ""
+		(property "Footprint" "aavirk:Resistor_1_4W"
 			(at 85.852 91.44 90)
 			(effects
@@
 				(path "/1421b1c5-d608-4702-afbd-6fccffd87076"
 					(reference "R2")
+					(unit 1)
+				)
+			)
+		)
+	)
+	(symbol
+		(lib_id "power:GNDREF")
+		(at 189.23 68.58 0)
+		(unit 1)
+		(exclude_from_sim no)
+		(in_bom yes)
+		(on_board yes)
+		(dnp no)
+		(fields_autoplaced yes)
+		(property "Reference" "#PWR05"
+			(at 189.23 74.93 0)
+			(effects
+				(font
+					(size 1.27 1.27)
+				)
+				(hide yes)
+			)
+		)
+		(property "Value" "GNDREF"
+			(at 189.23 73.66 0)
+			(effects
+				(font
+					(size 1.27 1.27)
+				)
+			)
+		)
+		(property "Footprint" ""
+			(at 189.23 68.58 0)
+			(effects
+				(font
+					(size 1.27 1.27)
+				)
+				(hide yes)
+			)
+		)
+		(property "Datasheet" ""
+			(at 189.23 68.58 0)
+			(effects
+				(font
+					(size 1.27 1.27)
+				)
+				(hide yes)
+			)
+		)
+		(property "Description" "Power symbol creates a global label with name \"GNDREF\" , reference supply ground"
+			(at 189.23 68.58 0)
+			(effects
+				(font
+					(size 1.27 1.27)
+				)
+				(hide yes)
+			)
+		)
+		(pin "1"
+		)
+		(instances
+			(project ""
+				(path "/1421b1c5-d608-4702-afbd-6fccffd87076"
+					(reference "#PWR05")
 					(unit 1)
 				)
@@
 			)
 		)
-		(property "Footprint" "Capacitor_THT:CP_Radial_D10.0mm_P5.00mm"
+		(property "Footprint" "aavirk:Capacitor_Eletrolítico_10mm"
 			(at 199.0852 63.5 0)
 			(effects
@@
 			)
 		)
-		(property "Footprint" ""
+		(property "Footprint" "aavirk:Conector KRE"
 			(at 209.55 96.52 0)
 			(effects
@@
 			)
 		)
-		(property "Footprint" "Capacitor_THT:CP_Radial_D10.0mm_P5.00mm"
+		(property "Footprint" "aavirk:Capacitor_Eletrolítico_7.5mm"
 			(at 200.66 90.4748 0)
 			(effects
@@
 			)
 		)
-		(property "Footprint" ""
+		(property "Footprint" "aavirk:Resistor_1_4W"
 			(at 163.83 89.408 90)
 			(effects
@@
 			)
 		)
-		(property "Footprint" "Capacitor_THT:CP_Radial_D10.0mm_P5.00mm"
+		(property "Footprint" "aavirk:Capacitor_Eletrolítico_7.5mm"
 			(at 60.96 91.1352 0)
 			(effects
@@
 			)
 		)
-		(property "Footprint" ""
+		(property "Footprint" "aavirk:Capacitor_Poliesterg"
 			(at 159.7152 63.5 0)
 			(effects
@@
 			)
 		)
-		(property "Footprint" ""
+		(property "Footprint" "aavirk:Capacitor_Eletrolítico_5mm"
 			(at 73.3552 85.09 0)
 			(effects
@@
 			)
 		)
-		(property "Footprint" ""
+		(property "Footprint" "aavirk:Capacitor_Poliesterp"
 			(at 73.3552 106.68 0)
 			(effects
@@
 			)
 		)
-		(property "Footprint" ""
+		(property "Footprint" "aavirk:Conector KRE"
 			(at 125.73 31.75 0)
 			(effects
@@
 			)
 		)
-		(property "Footprint" "Virk:LA4182"
+		(property "Footprint" "aavirk:Circuito integrado"
 			(at 133.35 82.55 0)
 			(effects
@@
 			)
 		)
-		(property "Footprint" ""
+		(property "Footprint" "aavirk:Capacitor_Poliesterg"
 			(at 97.4852 86.36 0)
 			(effects
@@
 			)
 		)
-		(property "Footprint" ""
+		(property "Footprint" "aavirk:Conector KRE"
 			(at 142.24 31.75 0)
 			(effects
@@
 			)
 		)
-		(property "Footprint" ""
+		(property "Footprint" "aavirk:Resistor_220_1_4W"
 			(at 183.642 54.61 90)
 			(effects
@@
 			)
 		)
-		(property "Footprint" "Capacitor_THT:CP_Radial_D10.0mm_P5.00mm"
+		(property "Footprint" "aavirk:Capacitor_Eletrolítico_5mm"
 			(at 88.5952 106.68 0)
 			(effects
@@
 			)
 		)
-		(property "Footprint" "Capacitor_THT:CP_Radial_D10.0mm_P5.00mm"
+		(property "Footprint" "aavirk:Capacitor_Eletrolítico_5mm"
 			(at 185.1152 91.44 0)
 			(effects
@@
 			)
 		)
-		(property "Footprint" ""
+		(property "Footprint" "aavirk:Potenciometro_dual"
 			(at 127 50.165 0)
 			(effects
@@
 			)
 		)
-		(property "Footprint" "LED_THT:LED_D5.0mm"
+		(property "Footprint" "aavirk:Led_5mm"
 			(at 182.626 63.754 0)
 			(effects
@@
 			)
 		)
-		(property "Footprint" ""
+		(property "Footprint" "aavirk:Capacitor_Poliesterp"
 			(at 185.1152 106.68 0)
 			(effects

Commit message: aaaaa
Connections:
- net GNDREF: now also J1.2 (Pin_2), J3.1 (Pin_1), J5.2 (Pin_2); no longer J1.1 (Pin_1), J3.2 (Pin_2), J5.1 (Pin_1)
- net at C7.1, IC1.12 (12/VCC), R1.1: now also J5.1 (Pin_1); no longer J5.2 (Pin_2)
- net at C1.2: now also J1.1 (Pin_1); no longer J1.2 (Pin_2)
- net at RV1.1: now also J3.2 (Pin_2); no longer J3.1 (Pin_1)
Other:
- moved on the sheet: J1, J3, J5
