File: kitcat/kitcat.kicad_pcb (KiCad board)
At the start: 2 copper layers, 52 x 61.5 mm, 23 parts, among them IC1 LA4182, J1 Conn_01x02, J2 Conn_01x02, J3 Conn_01x02, J4 Conn_01x02, J5 Conn_01x02

Commit message: hterhytnnnytjjyjnyt
Parts:
- added G***: LOGO, LOGO, F.Cu at (156.2, 106.5)
- added G***: LOGO, LOGO, F.Cu at (158.5, 63.0)
- moved J5 9.21 mm to (154.2, 72.3), turned to -90 degrees
- moved C4 8.97 mm to (162.2, 91.5)
- moved J1 8.74 mm to (154.5, 94.8)
- moved C5 7.50 mm to (167.0, 99.0), turned to 90 degrees
- moved J2 2.37 mm to (189.0, 100.0), turned to 90 degrees
- moved J3 1.73 mm to (165.5, 114.2), turned to 0 degrees
Routing:
- net Net-(J1-Pin_1): track 26.3 -> 10.7 mm
- net GNDREF: track 44.0 -> 29.3 mm
- net Net-(IC1-12/VCC): track 27.0 -> 40.5 mm
- net Net-(C4-Pad1): track 2.91 -> 15.7 mm
- net Net-(C5-Pad1): track 32.7 -> 23.7 mm
- net Net-(IC1-8/IN1): track 18.2 -> 10.9 mm
- net Net-(J2-Pin_2): track 17.0 -> 22.7 mm
- net Net-(IC1-5/IN2): track 5.51 -> 10.1 mm
- net Net-(J3-Pin_2): track 11.8 -> 8.54 mm
Other:
- board size 52 x 61.5 mm -> 46.5 x 59 mm

Commit message: yt
Parts:
- removed the G*** at (156.2, 106.5)
- removed the G*** at (158.5, 63.0)
- added G***: LOGO, LOGO, F.Cu at (191.7, 88.0)
- added G***: LOGO, LOGO, F.Cu at (160.5, 102.3)
- added G***: LOGO, LOGO, F.Cu at (181.7, 74.2)
- added G***: LOGO, LOGO, F.Cu at (173.4, 104.5)
- added G***: LOGO, LOGO, F.Cu at (158.7, 62.8)
- added G***: LOGO, LOGO, F.Cu at (193.8, 101.8)
- moved J3 6.88 mm to (172.4, 114.3)
- moved R3 6.10 mm to (182.0, 91.0), turned to -90 degrees
- moved RV1 5.45 mm to (186.9, 112.5)
- moved C7 1.41 mm to (172.0, 67.0), turned to -90 degrees
- moved C9 1.41 mm to (186.0, 92.0), turned to 180 degrees
- moved J2 0.60 mm to (188.4, 100.2)
- turned D1 to 180 degrees
Routing:
- net GNDREF: track 29.3 -> 0.00 mm
- net Net-(J2-Pin_2): track 22.7 -> 39.5 mm
- net Net-(IC1-12/VCC): track 40.5 -> 29.7 mm
- net Net-(C4-Pad1): track 15.7 -> 7.48 mm
- net Net-(C8-Pad1): track 14.4 -> 19.6 mm
- net Net-(IC1-9/NF1): track 4.41 -> 5.91 mm
- net Net-(J3-Pin_2): track 8.54 -> 7.07 mm
- net Net-(IC1-2/OUT2): track 16.6 -> 17.6 mm
- net Net-(IC1-5/IN2): track 10.1 -> 9.40 mm
- net Net-(D1-Pad2): track 5.75 -> 5.04 mm
- net Net-(J1-Pin_1): track 10.7 -> 11.4 mm
Other:
- board text added: "*Feito na terra, por humanos*"
- board text added: "{dblquote}Look at you hacker, a pathetic creature of meat and bone. How can you challenge a perfect, immortal machine?{dblquote}"
