File: kitcat/kitcat.kicad_pcb (KiCad board)
At the start: 2 copper layers, 46.5 x 59 mm, 29 parts, among them IC1 LA4182, J1 Conn_01x02, J2 Conn_01x02, J3 Conn_01x02, J4 Conn_01x02, J5 Conn_01x02

Commit message: fyj
Other:
- board size 46.5 x 59 mm -> 46.5 x 59.2 mm
Changed lines of the file:
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@@
 	)
 	(gr_line
-		(start 197 72)
-		(end 197 118)
+		(start 197 59)
+		(end 197 118.2)
 		(stroke
 			(width 0.05)
@@
 	)
 	(gr_line
-		(start 150.5 118)
+		(start 150.5 118.2)
 		(end 150.5 59)
 		(stroke
@@
 	)
 	(gr_line
-		(start 197 59)
-		(end 197 72)
-		(stroke
-			(width 0.05)
-			(type default)
-		)
-		(layer "Edge.Cuts")
-	)
-	(gr_line
-		(start 197 118)
-		(end 150.5 118)
+		(start 197 118.2)
+		(end 150.5 118.2)
 		(stroke
 			(width 0.05)
@@
 		(polygon
 			(pts
-				(xy 197 118) (xy 197 59) (xy 150.5 59) (xy 150.5 118)
+				(xy 197 118.2) (xy 197 59) (xy 150.5 59) (xy 150.5 118.2)
 			)
 		)

Commit message: thy
Parts:
- J1 InR: renamed from J1
- J2 InR: renamed from J2
- J3 InL: renamed from J3
- J4 OutL: renamed from J4
- J5 PWR: renamed from J5
Routing:
- net GNDREF: vias 0 -> 3
- net (no net): vias 3 -> 0
Changed lines of the file:
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@@
 		(model "${PROJETOEX3D}/R1K.STEP"
 			(offset
-				(xyz 0 0 0)
+				(xyz 0 0 1)
 			)
 			(scale
@@
 		(layer "F.Cu")
 		(at 172.4 114.35)
-		(property "Reference" "J3"
-			(at -1.8 -6.1 0)
+		(property "Reference" "J3 InL"
+			(at -2 -5.55 0)
 			(unlocked yes)
 			(layer "F.SilkS")
@@
 		)
 		(fp_text user "${REFERENCE}"
-			(at 0.06 -6.2 0)
+			(at -2 -5.55 0)
 			(unlocked yes)
 			(layer "F.Fab")
@@
 		(layer "F.Cu")
 		(at 193.3 67.5 90)
-		(property "Reference" "J4"
-			(at 5.8 -0.25 0)
+		(property "Reference" "J4 OutL"
+			(at -6.6 -0.7 0)
 			(unlocked yes)
 			(layer "F.SilkS")
@@
 			(layer "F.SilkS")
 		)
-		(fp_text user "${REFERENCE}"
-			(at -0.35 -0.8 90)
+		(fp_text user "J4 OutL"
+			(at -6.6 -0.7 0)
 			(unlocked yes)
 			(layer "F.Fab")
@@
 		(layer "F.Cu")
 		(at 154.2 72.35 -90)
-		(property "Reference" "J5"
-			(at -0.35 -5.7 0)
+		(property "Reference" "J5 PWR"
+			(at -0.35 -7.6 0)
 			(unlocked yes)
 			(layer "F.SilkS")
@@
 		)
 		(fp_text user "${REFERENCE}"
-			(at 0.06 -6.2 270)
+			(at -0.35 -7.65 0)
 			(unlocked yes)
 			(layer "F.Fab")
@@
 		(layer "F.Cu")
 		(at 188.45 100.25 90)
-		(property "Reference" "J2"
-			(at 0.4 -5.5 90)
+		(property "Reference" "J2 InR"
+			(at 4.15 5.55 0)
 			(unlocked yes)
 			(layer "F.SilkS")
@@
 		)
 		(fp_text user "${REFERENCE}"
-			(at 0 -6 90)
+			(at 3.95 5.55 0)
 			(unlocked yes)
 			(layer "F.Fab")
@@
 		(at 182 91 -90)
 		(property "Reference" "R3"
-			(at -2.15 -1.95 270)
+			(at -1.95 -1.95 270)
 			(unlocked yes)
 			(layer "F.SilkS")
@@
 		(layer "F.Cu")
 		(at 154.475 94.85 -90)
-		(property "Reference" "J1"
-			(at 6.15 -1.35 0)
+		(property "Reference" "J1 InR"
+			(at 6.25 0.575 0)
 			(unlocked yes)
 			(layer "F.SilkS")
@@
 		)
 		(fp_text user "${REFERENCE}"
-			(at 0.06 -6.2 270)
+			(at 5.95 0.875 0)
 			(unlocked yes)
 			(layer "F.Fab")
@@
 		)
 	)
-	(via
-		(at 193.723683 75.973143)
-		(size 0.6)
-		(drill 0.3)
-		(layers "F.Cu" "B.Cu")
-		(free yes)
-		(net 0)
-	)
-	(via
-		(at 157.432099 105.02182)
-		(size 0.6)
-		(drill 0.3)
-		(layers "F.Cu" "B.Cu")
-		(free yes)
-		(net 0)
-	)
-	(via
-		(at 163.673327 66.264567)
-		(size 0.6)
-		(drill 0.3)
-		(layers "F.Cu" "B.Cu")
-		(free yes)
-		(net 0)
-	)
 	(segment
 		(start 153 83)
@@
 		(net 3)
 	)
+	(via
+		(at 193.723683 75.973143)
+		(size 2)
+		(drill 1)
+		(layers "F.Cu" "B.Cu")
+		(free yes)
+		(net 4)
+	)
+	(via
+		(at 157.432099 105.02182)
+		(size 2)
+		(drill 1)
+		(layers "F.Cu" "B.Cu")
+		(free yes)
+		(net 4)
+	)
+	(via
+		(at 163.673327 66.264567)
+		(size 2)
+		(drill 1)
+		(layers "F.Cu" "B.Cu")
+		(free yes)
+		(net 4)
+	)
 	(segment
