File: kitcat/kitcat.kicad_pcb (KiCad board)
At the start: 2 copper layers, 46.5 x 59.2 mm, 29 parts, among them IC1 LA4182, J1 InR Conn_01x02, J2 InR Conn_01x02, J3 InL Conn_01x02, J4 OutL Conn_01x02, J5 PWR Conn_01x02

Commit message: nh
Other:
- board size 46.5 x 59.2 mm -> 48.5 x 61.5 mm
Changed lines of the file:
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@@
 		(pad "1" thru_hole circle
 			(at -5 0 270)
-			(size 2 2)
-			(drill 1)
+			(size 1.5 1.5)
+			(drill 0.8)
 			(layers "*.Cu" "*.Mask")
 			(remove_unused_layers no)
@@
 		(pad "2" thru_hole circle
 			(at 5 0 270)
-			(size 2 2)
-			(drill 1)
+			(size 1.5 1.5)
+			(drill 0.8)
 			(layers "*.Cu" "*.Mask")
 			(remove_unused_layers no)
@@
 			(layer "F.SilkS")
 		)
+		(fp_text user "${REFERENCE}"
+			(at 0.06 -6.2 90)
+			(unlocked yes)
+			(layer "F.Fab")
+			(effects
+				(font
+					(size 1 1)
+					(thickness 0.15)
+				)
+			)
+		)
 		(fp_text user "J4 OutL"
 			(at -6.6 -0.7 0)
@@
 			)
 			(scale
-				(xyz 0.9 1 1)
+				(xyz 0.95 0.95 0.95)
 			)
 			(rotate
-				(xyz 90 -180 -180)
+				(xyz 90 -180 -0)
 			)
 		)
@@
 			)
 			(rotate
-				(xyz 90 -180 -180)
+				(xyz 90 -180 -0)
 			)
 		)
@@
 			)
 			(rotate
-				(xyz 90 -180 -180)
+				(xyz 90 -180 -0)
 			)
 		)
@@
 			)
 			(rotate
-				(xyz 90 -180 -180)
+				(xyz 90 -180 -0)
 			)
 		)
@@
 			)
 			(rotate
-				(xyz 90 -180 -180)
+				(xyz 90 -180 -0)
 			)
 		)
@@
 			)
 			(scale
-				(xyz 0.9 1 1)
+				(xyz 0.95 0.95 0.95)
 			)
 			(rotate
-				(xyz 90 -180 -180)
+				(xyz 90 -180 -0)
 			)
 		)
@@
 			)
 			(rotate
-				(xyz -90 -0 -0)
+				(xyz -90 -0 180)
 			)
 		)
@@
 			)
 			(rotate
-				(xyz -90 -0 -0)
+				(xyz -90 -0 180)
 			)
 		)
@@
 			)
 			(rotate
-				(xyz 90 -180 -180)
+				(xyz 90 -180 -0)
 			)
 		)
 	)
 	(gr_line
-		(start 150.5 59)
-		(end 197 59)
+		(start 149.5 58)
+		(end 198 58)
 		(stroke
 			(width 0.05)
@@
 	)
 	(gr_line
-		(start 197 59)
-		(end 197 118.2)
+		(start 198 58)
+		(end 198 119.5)
 		(stroke
 			(width 0.05)
@@
 	)
 	(gr_line
-		(start 150.5 118.2)
-		(end 150.5 59)
+		(start 149.5 119.5)
+		(end 149.5 58)
 		(stroke
 			(width 0.05)
@@
 	)
 	(gr_line
-		(start 197 118.2)
-		(end 150.5 118.2)
+		(start 198 119.5)
+		(end 149.5 119.5)
 		(stroke
 			(width 0.05)
@@
 		(polygon
 			(pts
-				(xy 197 118.2) (xy 197 59) (xy 150.5 59) (xy 150.5 118.2)
+				(xy 198 119.2) (xy 198 58) (xy 149.5 58) (xy 149.5 119.2)
 			)
 		)
