File: kitcat/kitcat.kicad_sch (KiCad schematic)
At the start: 23 parts, among them IC1 LA4182, J1 Conn_01x02, J2 Conn_01x02, J3 Conn_01x02, J4 Conn_01x02, J5 Conn_01x02

Commit message: aerg
Parts:
- J1 InR: renamed from J1
- J2 InR: renamed from J2
- J3 InL: renamed from J3
- J4 OutL: renamed from J4
- J5 PWR: renamed from J5
Changed lines of the file:
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@@
 		(on_board yes)
 		(dnp no)
-		(property "Reference" "J5"
+		(property "Reference" "J5 PWR"
 			(at 223.266 60.96 0)
 			(effects
@@
 			(project "Projeto2025.2"
 				(path "/1421b1c5-d608-4702-afbd-6fccffd87076"
-					(reference "J5")
+					(reference "J5 PWR")
 					(unit 1)
 				)
@@
 		(on_board yes)
 		(dnp no)
-		(property "Reference" "J1"
+		(property "Reference" "J1 InR"
 			(at 53.34 105.41 0)
 			(effects
@@
 			(project ""
 				(path "/1421b1c5-d608-4702-afbd-6fccffd87076"
-					(reference "J1")
+					(reference "J1 InR")
 					(unit 1)
 				)
@@
 		(on_board yes)
 		(dnp no)
-		(property "Reference" "J4"
+		(property "Reference" "J4 OutL"
 			(at 211.836 96.52 0)
 			(effects
@@
 			(project "Projeto2025.2"
 				(path "/1421b1c5-d608-4702-afbd-6fccffd87076"
-					(reference "J4")
+					(reference "J4 OutL")
 					(unit 1)
 				)
@@
 		(on_board yes)
 		(dnp no)
-		(property "Reference" "J2"
+		(property "Reference" "J2 InR"
 			(at 125.476 26.67 90)
 			(effects
@@
 			(project ""
 				(path "/1421b1c5-d608-4702-afbd-6fccffd87076"
-					(reference "J2")
+					(reference "J2 InR")
 					(unit 1)
 				)
@@
 		(on_board yes)
 		(dnp no)
-		(property "Reference" "J3"
+		(property "Reference" "J3 InL"
 			(at 139.7 26.924 90)
 			(effects
@@
 			(project ""
 				(path "/1421b1c5-d608-4702-afbd-6fccffd87076"
-					(reference "J3")
-					(unit 1)
-				)
+					(reference "J3 InL")
+					(unit 1)
+				)
